File: hardware/t3/t3.sch (KiCad schematic (older format))
At the start: 4 parts

Commit message: fix[1/x] ubertooth debug board
Parts:
- removed U?: ADUC816, symbol ADUC816
- added C? (x4): 1nf, symbol C
- added C?: 10pf, symbol C
- added C?: 6p8, symbol C
- added C?: 1pf, symbol C
- added C?: 2p2, symbol C
- added C?: 18pf, symbol C
- added L?: 2n2, symbol INDUCTOR
- added L?: 3nH, symbol INDUCTOR
- added P?: SMA, symbol SMA-CONN
- added R?: 4k3, symbol R
- L1: renamed from L?; value L_Small -> NC
- gave numbers to parts that had none: 2
Connections:
- net labels added: +3.3V, GND, w123
- wire segments 3 -> 46
Other:
- note added: "tx line inductor\n"
- moved on the sheet: L1, U1, U2

Commit message: fix[2/x] ubertooth debug board
Parts:
- added C? (x3): 68pf, symbol C
- added C? (x2): 100nf, symbol C
- added C? (x2): 27pf, symbol C
- added C?: 10nf, symbol C
- added R?: 10k, symbol R
- added R?: 43k, symbol R
- added Y?: 16MHz, symbol Crystal
- renumbered L1 to L?, U2 to U?, U1 to U?
Connections:
- net labels added: +1V8, ATEST1, ATEST2, CSn, DCLK, DIO, GIO1, GIO6, GPIO3.3, GR, HGM, PAEN, RX, SCLK, SI, SO, TX
- net labels removed: w123
- wire segments 46 -> 112
- no-connect marks 0 -> 8
Other:
- moved on the sheet: C?

Commit message: fix[3/x] ubertooth debug board
Parts:
- added C? (x2): 100nf, symbol C
- added C? (x2): 2.2uf, symbol C
- added C? (x2): 22pf, symbol C
- added C? (x2): 6pf, symbol C
- added P?: USB_B, symbol USB_B
- added P?: CONN_02X03, symbol CONN_02X03
- added Q?: 9012, symbol Q_PNP_BEC
- added R? (x2): 22R, symbol R
- added R?: 1K5, symbol R
- added R?: 2k2, symbol R
- added R?: 10k, symbol R
- added R?: 100K, symbol R
- added R?: 0R, symbol R
- added R? (x2): 10K, symbol R
- added SW? (x2): SW_PUSH, symbol SW_PUSH
- added U?: STM32F405RGTx, LQFP64, symbol STM32F405RGTx
- added Y?: 16MHz, symbol Crystal
- added Y?: 32.768k, symbol Crystal
Connections:
- net labels added: BOOT0, BOOT1, NRST, USBEN, VBUS
- wire segments 112 -> 180

Commit message: fix[4/x] ubertooth debug board
Parts:
- removed C?: 100nf, symbol C
- added C25, C26, C29: 10uf, Capacitors_SMD:C_0402, symbol C
- added C27, C28, C30: 100nf, Capacitors_SMD:C_0402, symbol C
- added D1, D2, D3, D4: LED, Capacitors_SMD:C_0402, symbol LED
- added P3: UART1, Pin_Headers:Pin_Header_Straight_1x03, symbol CONN_01X03
- added P4: SWD, Pin_Headers:Pin_Header_Straight_1x04, symbol CONN_01X04
- added R1, R3, R4, R5: 330, Capacitors_SMD:C_0402, symbol R
- added U4: LM1117-3.3, TO_SOT_Packages_SMD:SOT-223, symbol LM1117-3.3
- added U5: LM1117-1.8, TO_SOT_Packages_SMD:SOT-223, symbol LM1117-3.3
- C1, C10, C11, C12, C13, C14, C15, C16, C17, C18, C19, C2, C20, C21, C22, C23, C24, C3, C4, C5, C6, C7, C8, C9: renamed from C?; footprint (none) -> Capacitors_SMD:C_0402
- L1, L2, L3: renamed from L?; footprint (none) -> Capacitors_SMD:C_0402
- P1: renamed from P?; footprint (none) -> w_conn_rf:lemo_epb00250ntn
- P2: renamed from P?; value CONN_02X03 -> CON; footprint (none) -> Pin_Headers:Pin_Header_Straight_2x03
- P5: renamed from P?; footprint (none) -> Connect:USB_Mini-B
- Q1: renamed from Q?; footprint (none) -> TO_SOT_Packages_SMD:SC-70
- R10, R11, R12, R13, R14, R15, R16, R2, R6, R7, R8, R9: renamed from R?; footprint (none) -> Capacitors_SMD:C_0402
- SW1, SW2: renamed from SW?; footprint (none) -> Buttons_Switches_SMD:SW_SPST_EVQPE1
- U1: renamed from U?; footprint (none) -> Housings_DFN_QFN:QFN-16-1EP_4x4mm_Pitch0.65mm
- U2: renamed from U?; footprint (none) -> Housings_DFN_QFN:QFN-48-1EP_7x7mm_Pitch0.5mm
- U3: renamed from U?; footprint LQFP64 -> Housings_QFP:LQFP-64_10x10mm_Pitch0.5mm
- Y1, Y3: renamed from Y?; footprint (none) -> Crystals:Crystal_HC48-U_Vertical
- Y2: renamed from Y?; footprint (none) -> Crystals:Crystal_Round_Horizontal_3mm
Connections:
- net +1V8: now also U5.3 (VI)
- net +3V3: now also P4.1 (P1), U4.3 (VI)
- net CSn: now also U3.20 (ADC1_IN4/ADC2_IN4/DAC_OUT1/I2S3_WS/SPI1_NSS/SPI3_NSS/USART2_CK/USB_OTG_HS_SOF/PA4)
- net DCLK: now also U3.55 (I2S3_CK/SPI1_SCK/SPI3_SCK/SYS_JTDO-SWO/TIM2_CH2/PB3)
- net DIO: now also U3.56 (I2S3_ext_SD/SPI1_MISO/SPI3_MISO/SYS_JTRST/TIM3_CH1/PB4), U3.57 (CAN2_RX/I2C1_SMBA/I2S3_SD/SPI1_MOSI/SPI3_MOSI/TIM3_CH2/USB_OTG_HS_ULPI_D7/PB5)
- net GND: now also C25.1, C26.1, C27.1, C28.1, C29.1, C30.1, D1.1 (K), D2.1 (K), D3.1 (K), D4.1 (K), P3.1 (P1), P4.4 (P4), U4.1 (GND/ADJ), U5.1 (GND/ADJ)
- net SCLK: now also U3.21 (ADC1_IN5/ADC2_IN5/DAC_OUT2/SPI1_SCK/TIM2_CH1/TIM2_ETR/TIM8_CH1N/USB_OTG_HS_ULPI_CK/PA5)
- net SI: now also U3.23 (ADC1_IN7/ADC2_IN7/SPI1_MOSI/TIM14_CH1/TIM1_CH1N/TIM3_CH2/TIM8_CH1N/PA7)
- net SO: now also U3.22 (ADC1_IN6/ADC2_IN6/SPI1_MISO/TIM13_CH1/TIM1_BKIN/TIM3_CH1/TIM8_BKIN/PA6)
- net VBUS: now also U4.2 (VO), U4.4 (VO), U5.2 (VO), U5.4 (VO)
- net UAER1_TX: now reaches U3.42 (DAC_EXTI9/I2C3_SMBA/TIM1_CH2/USART1_TX/USB_OTG_FS_VBUS/PA9)
- net UAER1_TX: now also P3.2 (P2)
- net UAER1_RX: now reaches U3.43 (TIM1_CH3/USART1_RX/USB_OTG_FS_ID/PA10)
- net UAER1_RX: now also P3.3 (P3)
- net at U3.46 (SYS_JTMS-SWDIO/PA13): now also P4.2 (P2)
- net at U3.49 (SYS_JTCK-SWCLK/PA14): now also P4.3 (P3)
- new net: D1.2 (A), R1.2
- new net: D2.2 (A), R3.2
- new net: D3.2 (A), R4.2
- new net: D4.2 (A), R5.2
Other:
- note added: "->"
- note added: "Embedded bootloader\n• USART1 (PA9/PA10)\n• USART3 (PB10/11 and PC10/11)"
- moved on the sheet: C1, C10, C11, C12, C13, C14, C15, C16, C17, C18, C19, C2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

Commit message: fix[5/x] ubertooth debug board
Connections:
- net +1V8: now also C26.2, C28.2, U5.2 (VO), U5.4 (VO); no longer U5.3 (VI)
- net +3V3: now also C25.1, C27.1, U4.2 (VO), U4.4 (VO); no longer U4.3 (VI)
- net GND: now also C25.2, C27.2; no longer C25.1, C27.1
- net VBUS: now also C29.2, C30.2, U4.3 (VI), U5.3 (VI); no longer U4.2 (VO), U4.4 (VO), U5.2 (VO), U5.4 (VO)
Other:
- moved on the sheet: C25, C26, C27, C28, U4, U5
Changed lines of the file:
@@
 F 3 "" H 10600 2800 50  0000 C CNN
 	1    10600 2800
-	1    0    0    -1
+	-1   0    0    1
 $EndComp
 Wire Wire Line
@@
 L GND #PWR049
 U 1 1 582BA641
-P 10600 3150
-F 0 "#PWR049" H 10600 2900 50  0001 C CNN
-F 1 "GND" H 10750 3100 50  0000 C CNN
-F 2 "" H 10600 3150 50  0000 C CNN
-F 3 "" H 10600 3150 50  0000 C CNN
-	1    10600 3150
-	1    0    0    -1
+P 10600 2450
+F 0 "#PWR049" H 10600 2200 50  0001 C CNN
+F 1 "GND" H 10750 2400 50  0000 C CNN
+F 2 "" H 10600 2450 50  0000 C CNN
+F 3 "" H 10600 2450 50  0000 C CNN
+	1    10600 2450
+	1    0    0    1
 $EndComp
 Wire Wire Line
-	10600 3150 10600 3100
+	10600 2450 10600 2500
 Connection ~ 11200 2800
 $Comp
@@
 L C C25
 U 1 1 582C1592
-P 9850 2950
-F 0 "C25" V 9750 3050 50  0000 L CNN
-F 1 "10uf" V 9950 2800 50  0000 L CNN
-F 2 "Capacitors_SMD:C_0402" H 9888 2800 50  0001 C CNN
-F 3 "" H 9850 2950 50  0000 C CNN
-	1    9850 2950
+P 9850 2650
+F 0 "C25" V 9750 2750 50  0000 L CNN
+F 1 "10uf" V 9950 2500 50  0000 L CNN
+F 2 "Capacitors_SMD:C_0402" H 9888 2500 50  0001 C CNN
+F 3 "" H 9850 2650 50  0000 C CNN
+	1    9850 2650
 	-1   0    0    1
 $EndComp
@@
 L C C27
 U 1 1 582C1598
-P 10100 2950
-F 0 "C27" V 10000 3050 50  0000 L CNN
-F 1 "100nf" V 10200 2800 50  0000 L CNN
-F 2 "Capacitors_SMD:C_0402" H 10138 2800 50  0001 C CNN
-F 3 "" H 10100 2950 50  0000 C CNN
-	1    10100 2950
+P 10100 2650
+F 0 "C27" V 10000 2750 50  0000 L CNN
+F 1 "100nf" V 10200 2500 50  0000 L CNN
+F 2 "Capacitors_SMD:C_0402" H 10138 2500 50  0001 C CNN
+F 3 "" H 10100 2650 50  0000 C CNN
+	1    10100 2650
 	-1   0    0    1
 $EndComp
 Wire Wire Line
-	9850 3100 9850 3150
+	9850 2500 9850 2450
 Wire Wire Line
-	10100 3150 10100 3100
+	10100 2450 10100 2500
 Wire Wire Line
-	9850 3150 10600 3150
-Connection ~ 10100 3150
+	9850 2450 10600 2450
+Connection ~ 10100 2450
 $Comp
 L LM1117-3.3 U5
@@
 F 3 "" H 10600 3600 50  0000 C CNN
 	1    10600 3600
-	1    0    0    -1
+	-1   0    0    1
 $EndComp
 $Comp
 L GND #PWR051
 U 1 1 582C2901
-P 10600 3950
-F 0 "#PWR051" H 10600 3700 50  0001 C CNN
-F 1 "GND" H 10750 3900 50  0000 C CNN
-F 2 "" H 10600 3950 50  0000 C CNN
-F 3 "" H 10600 3950 50  0000 C CNN
-	1    10600 3950
-	1    0    0    -1
+P 10600 3250
+F 0 "#PWR051" H 10600 3000 50  0001 C CNN
+F 1 "GND" H 10750 3200 50  0000 C CNN
+F 2 "" H 10600 3250 50  0000 C CNN
+F 3 "" H 10600 3250 50  0000 C CNN
+	1    10600 3250
+	1    0    0    1
 $EndComp
 Wire Wire Line
-	10600 3950 10600 3900
+	10600 3250 10600 3300
 Wire Wire Line
 	9600 3600 10300 3600
@@
 L C C26
 U 1 1 582C2909
-P 9850 3750
-F 0 "C26" V 9750 3850 50  0000 L CNN
-F 1 "10uf" V 9950 3600 50  0000 L CNN
-F 2 "Capacitors_SMD:C_0402" H 9888 3600 50  0001 C CNN
-F 3 "" H 9850 3750 50  0000 C CNN
-	1    9850 3750
-	-1   0    0    1
+P 9850 3450
+F 0 "C26" V 9750 3550 50  0000 L CNN
+F 1 "10uf" V 9950 3300 50  0000 L CNN
+F 2 "Capacitors_SMD:C_0402" H 9888 3300 50  0001 C CNN
+F 3 "" H 9850 3450 50  0000 C CNN
+	1    9850 3450
+	-1   0    0    -1
 $EndComp
 $Comp
 L C C28
 U 1 1 582C290F
-P 10100 3750
-F 0 "C28" V 10000 3850 50  0000 L CNN
-F 1 "100nf" V 10200 3600 50  0000 L CNN
-F 2 "Capacitors_SMD:C_0402" H 10138 3600 50  0001 C CNN
-F 3 "" H 10100 3750 50  0000 C CNN
-	1    10100 3750
-	-1   0    0    1
+P 10100 3450
+F 0 "C28" V 10000 3550 50  0000 L CNN
+F 1 "100nf" V 10200 3300 50  0000 L CNN
+F 2 "Capacitors_SMD:C_0402" H 10138 3300 50  0001 C CNN
+F 3 "" H 10100 3450 50  0000 C CNN
+	1    10100 3450
+	-1   0    0    -1
 $EndComp
 Wire Wire Line
-	9850 3900 9850 3950
+	9850 3300 9850 3250
 Wire Wire Line
-	10100 3950 10100 3900
+	10100 3250 10100 3300
 Wire Wire Line
-	9850 3950 10600 3950
-Connection ~ 10100 3950
+	9850 3250 10600 3250
+Connection ~ 10100 3250
 Wire Wire Line
 	11200 3600 10900 3600
@@
 	0    -1   -1   0
 $EndComp
+Connection ~ 9850 2800
+Connection ~ 10100 2800
+Connection ~ 11350 2800
+Connection ~ 11600 2800
+Connection ~ 9850 3600
+Connection ~ 10100 3600
 $EndSCHEMATC

Commit message: fix[6/x] ubertooth debug board
Parts:
- C1, C10, C11, C12, C13, C14, C15, C16, C17, C18, C19, C2, C20, C21, C22, C23, C24, C25, C26, C27, C28, C29, C3, C30, C4, C5, C6, C7, C8, C9, D1, D2, D3, D4, L1, L2, L3, R1, R10, R11, R12, R13, R14, R15, R16, R2, R3, R4, R5, R6, R7, R8, R9: footprint Capacitors_SMD:C_0402 -> Capacitors_SMD:C_0603_HandSoldering
- Q1: footprint TO_SOT_Packages_SMD:SC-70 -> TO_SOT_Packages_SMD:SOT-23
- Y1, Y3: footprint Crystals:Crystal_HC48-U_Vertical -> Crystals:Crystal_HC50-U_Vertical

Commit message: update[7/x] ubertooth debug board
Parts:
- added R17, R18: 0R, Capacitors_SMD:C_0603_HandSoldering, symbol R
- C17, C4, C6: footprint Capacitors_SMD:C_0603_HandSoldering -> Capacitors_SMD:C_0805_HandSoldering
Connections:
- net +3V3: now also C16.1, U1.1 (AVDD_PA1), R17.2
- net ATEST1: now also U3.15 (ADC1_IN1/ADC2_IN1/ADC3_IN1/TIM2_CH2/TIM5_CH2/UART4_RX/USART2_RTS/PA1)
- net ATEST2: now also U3.16 (ADC1_IN2/ADC2_IN2/ADC3_IN2/TIM2_CH3/TIM5_CH3/TIM9_CH1/USART2_TX/PA2)
- net GIO1: now also U3.34 (CAN2_TX/I2S2_CK/SPI2_SCK/TIM1_CH1N/USART3_CTS/USB_OTG_HS_ULPI_D6/USB_OTG_HS_VBUS/PB13)
- net GIO6: now also U3.17 (ADC1_IN3/ADC2_IN3/ADC3_IN3/TIM2_CH4/TIM5_CH4/TIM9_CH2/USART2_RX/USB_OTG_HS_ULPI_D0/PA3)
- net GPIO3.3: now also U3.33 (CAN2_RX/I2C2_SMBA/I2S2_WS/SPI2_NSS/TIM1_BKIN/USART3_CK/USB_OTG_HS_ID/USB_OTG_HS_ULPI_D5/PB12), R18.1; no longer U2.25 (DVDD3.3)
- net GR: now also U3.35 (I2S2_ext_SD/SPI2_MISO/TIM12_CH1/TIM1_CH2N/TIM8_CH2N/USART3_RTS/USB_OTG_HS_DM/PB14)
- net HGM: now also U3.10 (PC2/ADC1_IN12/ADC2_IN12/ADC3_IN12/I2S2_ext_SD/SPI2_MISO/USB_OTG_HS_ULPI_DIR)
- net PAEN: now also U3.11 (PC3/ADC1_IN13/ADC2_IN13/ADC3_IN13/I2S2_SD/SPI2_MOSI/USB_OTG_HS_ULPI_NXT)
- net RX: now also U3.30 (ADC1_EXTI11/ADC2_EXTI11/ADC3_EXTI11/I2C2_SDA/TIM2_CH4/USART3_RX/USB_OTG_HS_ULPI_D4/PB11)
- net TX: now also U3.29 (I2C2_SCL/I2S2_CK/SPI2_SCK/TIM2_CH3/USART3_TX/USB_OTG_HS_ULPI_D3/PB10)
- new net: R17.1, R18.2, U2.25 (DVDD3.3)
- no-connect marks 8 -> 23

Commit message: update
Parts:
- removed C23: 68pf, Capacitors_SMD:C_0603_HandSoldering, symbol C
- added D5: LED, Capacitors_SMD:C_0603_HandSoldering, symbol LED
- added R14: 330, Capacitors_SMD:C_0603_HandSoldering, symbol R
- C23: renamed from C24; footprint Capacitors_SMD:C_0603_HandSoldering -> Capacitors_SMD:C_0805_HandSoldering
- C24: renamed from C25; footprint Capacitors_SMD:C_0603_HandSoldering -> Capacitors_SMD:C_0805_HandSoldering
- C25: renamed from C26; footprint Capacitors_SMD:C_0603_HandSoldering -> Capacitors_SMD:C_0805_HandSoldering
- C28: renamed from C29; footprint Capacitors_SMD:C_0603_HandSoldering -> Capacitors_SMD:C_0805_HandSoldering
- R12: renamed from R17; value 0R -> 0R(NC)
- renumbered C27 to C26, C28 to C27, C30 to C29, R18 to R13, R12 to R15, R13 to R16, R14 to R17, R15 to R18, R16 to R19
Connections:
- net GND: now also D5.1 (K)
- net USBEN: now also U3.62 (CAN1_TX/DAC_EXTI9/I2C1_SDA/I2S2_WS/SDIO_D5/SPI2_NSS/TIM11_CH1/TIM4_CH4/PB9)
- net VBUS: now also R14.1; no longer U5.3 (VI)
- net LED4: now reaches U3.36 (ADC1_EXTI15/ADC2_EXTI15/ADC3_EXTI15/I2S2_SD/RTC_REFIN/SPI2_MOSI/TIM12_CH2/TIM1_CH3N/TIM8_CH3N/USB_OTG_HS_DP/PB15)
- net LED4: now also R5.1
- net LED3: now reaches U3.37 (PC6/I2S2_MCK/SDIO_D6/TIM3_CH1/TIM8_CH1/USART6_TX)
- net LED3: now also R4.1
- net LED2: now reaches U3.38 (PC7/I2S3_MCK/SDIO_D7/TIM3_CH2/TIM8_CH2/USART6_RX)
- net LED2: now also R3.1
- net LED1: now reaches U3.39 (PC8/SDIO_D0/TIM3_CH3/TIM8_CH3/USART6_CK)
- net LED1: now also R1.1
- new net: D5.2 (A), R14.2
- no-connect marks 23 -> 16
Changed lines of the file:
@@
 NoConn ~ 6850 1650
 NoConn ~ 6950 1650
-$Comp
-L C C23
-U 1 1 5824DF6C
-P 6850 1050
-F 0 "C23" V 6750 1150 50  0000 L CNN
-F 1 "68pf" V 6950 900 50  0000 L CNN
-F 2 "Capacitors_SMD:C_0603_HandSoldering" H 6888 900 50  0001 C CNN
-F 3 "" H 6850 1050 50  0000 C CNN
-	1    6850 1050
-	-1   0    0    1
-$EndComp
 NoConn ~ 7750 2450
 Text Label 4000 1150 2    60   Italic 12
@@
 GIO1
 $Comp
-L C C24
+L C C23
 U 1 1 5825965F
 P 7850 4550
-F 0 "C24" H 7875 4650 50  0000 L CNN
+F 0 "C23" H 7875 4650 50  0000 L CNN
 F 1 "100nf" H 7900 4450 50  0000 L CNN
-F 2 "Capacitors_SMD:C_0603_HandSoldering" H 7888 4400 50  0001 C CNN
+F 2 "Capacitors_SMD:C_0805_HandSoldering" H 7888 4400 50  0001 C CNN
 F 3 "" H 7850 4550 50  0000 C CNN
 	1    7850 4550
@@
 $EndComp
 $Comp
-L R R14
+L R R17
 U 1 1 5825807F
 P 14550 7300
-F 0 "R14" V 14650 7300 50  0000 C CNN
+F 0 "R17" V 14650 7300 50  0000 C CNN
 F 1 "22R" V 14550 7300 50  0000 C CNN
 F 2 "Capacitors_SMD:C_0603_HandSoldering" V 14480 7300 50  0001 C CNN
@@
 $EndComp
 $Comp
-L R R15
+L R R18
 U 1 1 58259354
 P 14550 7400
-F 0 "R15" V 14450 7400 50  0000 C CNN
+F 0 "R18" V 14450 7400 50  0000 C CNN
 F 1 "22R" V 14550 7400 50  0000 C CNN
 F 2 "Capacitors_SMD:C_0603_HandSoldering" V 14480 7400 50  0001 C CNN
@@
 $EndComp
 $Comp
-L R R16
+L R R19
 U 1 1 5825A6F7
 P 14800 7650
-F 0 "R16" V 14700 7650 50  0000 C CNN
+F 0 "R19" V 14700 7650 50  0000 C CNN
 F 1 "1K5" V 14800 7650 50  0000 C CNN
 F 2 "Capacitors_SMD:C_0603_HandSoldering" V 14730 7650 50  0001 C CNN
@@
 $EndComp
 $Comp
-L R R12
+L R R15
 U 1 1 5825B206
 P 14250 8100
-F 0 "R12" V 14150 8100 50  0000 C CNN
+F 0 "R15" V 14150 8100 50  0000 C CNN
 F 1 "2k2" V 14250 8100 50  0000 C CNN
 F 2 "Capacitors_SMD:C_0603_HandSoldering" V 14180 8100 50  0001 C CNN
@@
 $EndComp
 $Comp
-L R R13
+L R R16
 U 1 1 5825B29F
 P 14450 8300
-F 0 "R13" V 14350 8300 50  0000 C CNN
+F 0 "R16" V 14350 8300 50  0000 C CNN
 F 1 "10k" V 14450 8300 50  0000 C CNN
 F 2 "Capacitors_SMD:C_0603_HandSoldering" V 14380 8300 50  0001 C CNN
@@
 $EndComp
 $Comp
-L C C29
+L C C28
 U 1 1 582BD473
 P 11350 2950
-F 0 "C29" V 11250 3050 50  0000 L CNN
+F 0 "C28" V 11250 3050 50  0000 L CNN
 F 1 "10uf" V 11450 2800 50  0000 L CNN
-F 2 "Capacitors_SMD:C_0603_HandSoldering" H 11388 2800 50  0001 C CNN
+F 2 "Capacitors_SMD:C_0805_HandSoldering" H 11388 2800 50  0001 C CNN
 F 3 "" H 11350 2950 50  0000 C CNN
 	1    11350 2950
@@
 $EndComp
 $Comp
-L C C30
+L C C29
 U 1 1 582BD839
 P 11600 2950
-F 0 "C30" V 11500 3050 50  0000 L CNN
+F 0 "C29" V 11500 3050 50  0000 L CNN
 F 1 "100nf" V 11700 2800 50  0000 L CNN
 F 2 "Capacitors_SMD:C_0603_HandSoldering" H 11638 2800 50  0001 C CNN
@@
 VBUS
 $Comp
-L C C25
+L C C24
 U 1 1 582C1592
 P 9850 2650
-F 0 "C25" V 9750 2750 50  0000 L CNN
+F 0 "C24" V 9750 2750 50  0000 L CNN
 F 1 "10uf" V 9950 2500 50  0000 L CNN
-F 2 "Capacitors_SMD:C_0603_HandSoldering" H 9888 2500 50  0001 C CNN
+F 2 "Capacitors_SMD:C_0805_HandSoldering" H 9888 2500 50  0001 C CNN
 F 3 "" H 9850 2650 50  0000 C CNN
 	1    9850 2650
@@
 $EndComp
 $Comp
-L C C27
+L C C26
 U 1 1 582C1598
 P 10100 2650
-F 0 "C27" V 10000 2750 50  0000 L CNN
+F 0 "C26" V 10000 2750 50  0000 L CNN
 F 1 "100nf" V 10200 2500 50  0000 L CNN
 F 2 "Capacitors_SMD:C_0603_HandSoldering" H 10138 2500 50  0001 C CNN
@@
 $EndComp
 $Comp
-L C C26
+L C C25
 U 1 1 582C2909
 P 9850 3450
-F 0 "C26" V 9750 3550 50  0000 L CNN
+F 0 "C25" V 9750 3550 50  0000 L CNN
 F 1 "10uf" V 9950 3300 50  0000 L CNN
-F 2 "Capacitors_SMD:C_0603_HandSoldering" H 9888 3300 50  0001 C CNN
+F 2 "Capacitors_SMD:C_0805_HandSoldering" H 9888 3300 50  0001 C CNN
 F 3 "" H 9850 3450 50  0000 C CNN
 	1    9850 3450
@@
 $EndComp
 $Comp
-L C C28
+L C C27
 U 1 1 582C290F
 P 10100 3450
-F 0 "C28" V 10000 3550 50  0000 L CNN
+F 0 "C27" V 10000 3550 50  0000 L CNN
 F 1 "100nf" V 10200 3300 50  0000 L CNN
 F 2 "Capacitors_SMD:C_0603_HandSoldering" H 10138 3300 50  0001 C CNN
@@
 	0    -1   -1   0
 $EndComp
+NoConn ~ 12850 7700
+NoConn ~ 12850 7900
+NoConn ~ 12850 8000
+NoConn ~ 12850 8500
+NoConn ~ 12850 8600
+NoConn ~ 12850 8700
+$Comp
+L R R12
+U 1 1 5830C348
+P 7950 3750
+F 0 "R12" V 8030 3750 50  0000 C CNN
+F 1 "0R(NC)" V 7950 3750 50  0000 C CNN
+F 2 "Capacitors_SMD:C_0603_HandSoldering" V 7880 3750 50  0001 C CNN
+F 3 "" H 7950 3750 50  0000 C CNN
+	1    7950 3750
+	1    0    0    -1
+$EndComp
+$Comp
+L +3.3V #PWR054
+U 1 1 5830CDFB
+P 7950 3950
+F 0 "#PWR054" H 7950 3800 50  0001 C CNN
+F 1 "+3.3V" H 7800 3950 50  0000 C CNN
+F 2 "" H 7950 3950 50  0000 C CNN
+F 3 "" H 7950 3950 50  0000 C CNN
+	1    7950 3950
+	-1   0    0    1
+$EndComp
+$Comp
+L R R13
+U 1 1 5830D8CF
+P 8150 3550
+F 0 "R13" V 8230 3550 50  0000 C CNN
+F 1 "0R" V 8150 3550 50  0000 C CNN
+F 2 "Capacitors_SMD:C_0603_HandSoldering" V 8080 3550 50  0001 C CNN
+F 3 "" H 8150 3550 50  0000 C CNN
+	1    8150 3550
+	0    1    1    0
+$EndComp
+NoConn ~ 13250 6200
+NoConn ~ 12850 7000
+$Comp
+L LED D5
+U 1 1 582F3C21
+P 11200 4250
+F 0 "D5" H 11200 4350 50  0000 C CNN
+F 1 "LED" H 11200 4150 50  0000 C CNN
+F 2 "Capacitors_SMD:C_0603_HandSoldering" H 11200 4250 50  0001 C CNN
+F 3 "" H 11200 4250 50  0000 C CNN
+	1    11200 4250
+	0    -1   -1   0
+$EndComp
+$Comp
+L R R14
+U 1 1 582F3C27
+P 11200 3850
+F 0 "R14" V 11280 3850 50  0000 C CNN
+F 1 "330" V 11200 3850 50  0000 C CNN
+F 2 "Capacitors_SMD:C_0603_HandSoldering" V 11130 3850 50  0001 C CNN
+F 3 "" H 11200 3850 50  0000 C CNN
+	1    11200 3850
+	1    0    0    -1
+$EndComp
+$Comp
+L GND #PWR055
+U 1 1 582F3C2D
+P 11200 4500
+F 0 "#PWR055" H 11200 4250 50  0001 C CNN
+F 1 "GND" H 11200 4350 50  0000 C CNN
+F 2 "" H 11200 4500 50  0000 C CNN
+F 3 "" H 11200 4500 50  0000 C CNN
+	1    11200 4500
+	1    0    0    -1
+$EndComp
+Text Label 1200 7700 3    47   Italic 9
+LED1
+Text Label 1500 7700 3    47   Italic 9
+LED2
+Text Label 1800 7700 3    47   Italic 9
+LED3
+Text Label 2050 7700 3    47   Italic 9
+LED4
+Text Label 3950 8700 0    47   Italic 9
+LED1
+Text Label 3950 8600 0    47   Italic 9
+LED2
+Text Label 3950 8500 0    47   Italic 9
+LED3
+Text Label 13250 9400 2    47   Italic 9
+LED4
 Wire Wire Line
 	4500 3050 5050 3050
@@
 	6250 900  6250 850
 Wire Wire Line
-	6250 850  6850 850
-Wire Wire Line
 	6550 850  6550 900
 Wire Wire Line
@@
 Wire Wire Line
 	6550 1650 6550 1600
-Wire Wire Line
-	4950 1600 6850 1600
-Wire Wire Line
-	6850 1600 6850 1200
 Wire Wire Line
 	5850 1650 5850 1600
@@
 Connection ~ 5850 1600
 Connection ~ 4950 1600
-Wire Wire Line
-	6850 850  6850 900
 Connection ~ 6550 850
 Wire Wire Line
@@
 	1200 8650 1200 8700
 Wire Wire Line
-	1200 7900 1200 7800
+	1200 7700 1200 7900
 Wire Wire Line
 	1500 8200 1500 8250
@@
 	1500 8650 1500 8700
 Wire Wire Line
-	1500 7900 1500 7800
+	1500 7700 1500 7900
 Wire Wire Line
 	1800 8200 1800 8250
@@
 	1800 8650 1800 8700
 Wire Wire Line
-	1800 7900 1800 7800
+	1800 7700 1800 7900
 Wire Wire Line
 	2050 8200 2050 8250
@@
 	2050 8650 2050 8700
 Wire Wire Line
-	2050 7900 2050 7800
+	2050 7700 2050 7900
 Wire Wire Line
 	10900 2800 11850 2800
 Wire Wire Line
-	11200 2800 11200 3600
+	11200 2800 11200 3700
 Wire Wire Line
 	10600 2450 10600 2500
@@
 Wire Wire Line
 	4250 8200 3950 8200
-NoConn ~ 1200 7800
-NoConn ~ 1500 7800
-NoConn ~ 1800 7800
-NoConn ~ 2000 7800
-NoConn ~ 2050 7800
 Wire Wire Line
 	3550 7150 3850 7150
@@
 	3700 7200 3700 7150
 Connection ~ 3700 7150
-NoConn ~ 12850 7700
-NoConn ~ 12850 7900
-NoConn ~ 12850 8000
-NoConn ~ 12850 8500
-NoConn ~ 12850 8600
-NoConn ~ 12850 8700
-NoConn ~ 12850 8800
-NoConn ~ 12850 9400
-$Comp
-L R R17
-U 1 1 5830C348
-P 7950 3750
-F 0 "R17" V 8030 3750 50  0000 C CNN
-F 1 "0R" V 7950 3750 50  0000 C CNN
-F 2 "Capacitors_SMD:C_0603_HandSoldering" V 7880 3750 50  0001 C CNN
-F 3 "" H 7950 3750 50  0000 C CNN
-	1    7950 3750
-	1    0    0    -1
-$EndComp
 Wire Wire Line
 	7950 3600 7950 3550
@@
 Wire Wire Line
 	7950 3900 7950 3950
-$Comp
-L +3.3V #PWR054
-U 1 1 5830CDFB
-P 7950 3950
-F 0 "#PWR054" H 7950 3800 50  0001 C CNN
-F 1 "+3.3V" H 7800 3950 50  0000 C CNN
-F 2 "" H 7950 3950 50  0000 C CNN
-F 3 "" H 7950 3950 50  0000 C CNN
-	1    7950 3950
-	-1   0    0    1
-$EndComp
-$Comp
-L R R18
-U 1 1 5830D8CF
-P 8150 3550
-F 0 "R18" V 8230 3550 50  0000 C CNN
-F 1 "0R" V 8150 3550 50  0000 C CNN
-F 2 "Capacitors_SMD:C_0603_HandSoldering" V 8080 3550 50  0001 C CNN
-F 3 "" H 8150 3550 50  0000 C CNN
-	1    8150 3550
-	0    1    1    0
-$EndComp
 Wire Wire Line
 	7750 3550 8000 3550
 Wire Wire Line
 	8300 3550 8600 3550
-NoConn ~ 13250 6200
-NoConn ~ 12850 7000
+Wire Wire Line
+	6250 850  6550 850
+Wire Wire Line
+	6550 1600 4950 1600
+Wire Wire Line
+	11200 4000 11200 4050
+Wire Wire Line
+	11200 4450 11200 4500
+Wire Wire Line
+	12850 9400 13250 9400
+Wire Wire Line
+	4250 8500 3950 8500
+Wire Wire Line
+	4250 8600 3950 8600
+Wire Wire Line
+	4250 8700 3950 8700
+Wire Wire Line
+	12850 8800 13250 8800
+Text Label 13250 8800 2    47   Italic 9
+USBEN
 $EndSCHEMATC
