File: hardware/t3/t3.sch (KiCad schematic (older format))
At the start: 72 parts, among them P1 SMA, P2 CON, P3 UART1, P4 SWD, P5 USB_B, Q1 9012, SW1 SW_PUSH, SW2 SW_PUSH, U1 CC2591, U2 CC2400, U3 STM32F405RGTx, U4 LM1117-3.3, U5 LM1117-1.8, Y1 16MHz, Y2 32.768k, Y3 16MHz

Commit message: update[8/x] add logo & fix layout
Parts:
- added C30: 2.2pf, Capacitors_SMD:C_0603_HandSoldering, symbol C
- added L4: 1Kohms, Capacitors_SMD:C_0603_HandSoldering, symbol INDUCTOR
- added P6: power, Pin_Headers:Pin_Header_Straight_1x02, symbol CONN_01X02
- added P7: UART2, Pin_Headers:Pin_Header_Straight_1x03, symbol CONN_01X03
- added P8: Debug, Pin_Headers:Pin_Header_Straight_1x05, symbol CONN_01X05
- added t1, t2, t3, t4, t5, t6: TST, t3:test_pin, symbol TST
- Y1, Y3: footprint Crystals:Crystal_HC50-U_Vertical -> Crystals:Crystal_HC49-U_Vertical
Connections:
- net +3V3: now also L4.2; no longer C15.1, C16.1, C2.2, C4.2, C6.1, C7.1, P4.1 (P1), SW1.2, U1.1 (AVDD_PA1), U1.10 (AVDD_PA2), U1.13 (AVDD_LNA), U1.16 (AVDD_BIAS)
- net ATEST1: now also t1.1
- net ATEST2: now also t2.1
- net BOOT0: now also SW1.2; no longer SW1.1
- net DCLK: now also t6.1
- net DIO: now also t5.1
- net GIO1: now also t3.1
- net GIO6: now also t4.1
- net GND: now also C30.2, P6.2 (P2), P7.1 (P1)
- net VBUS: now also U5.3 (VI), P6.1 (P1)
- net debug4: now reaches U3.50 (ADC1_EXTI15/ADC2_EXTI15/ADC3_EXTI15/I2S3_WS/SPI1_NSS/SPI3_NSS/SYS_JTDI/TIM2_CH1/TIM2_ETR/PA15)
- net debug4: now also P8.1 (P1)
- net UAER2_TX: now reaches U3.51 (PC10/I2S3_CK/SDIO_D2/SPI3_SCK/UART4_TX/USART3_TX)
- net UAER2_TX: now also P7.3 (P3)
- net UAER2_RX: now reaches U3.52 (PC11/ADC1_EXTI11/ADC2_EXTI11/ADC3_EXTI11/I2S3_ext_SD/SDIO_D3/SPI3_MISO/UART4_RX/USART3_RX)
- net UAER2_RX: now also P7.2 (P2)
- net debug5: now reaches U3.54 (PD2/SDIO_CMD/TIM3_ETR/UART5_RX)
- net debug5: now also P8.2 (P2)
- net debug1: now reaches U3.58 (CAN2_TX/I2C1_SCL/TIM4_CH1/USART1_TX/PB6)
- net debug1: now also P8.3 (P3)
- net debug2: now reaches U3.59 (I2C1_SDA/TIM4_CH2/USART1_RX/PB7)
- net debug2: now also P8.4 (P4)
- net debug3: now reaches U3.61 (CAN1_RX/I2C1_SCL/SDIO_D4/TIM10_CH1/TIM4_CH3/PB8)
- net debug3: now also P8.5 (P5)
- new net +3.3VADC: C15.1, C16.1, C2.2, C30.1, C4.2, C6.1, C7.1, L4.1, P4.1 (P1), SW1.1, U1.1 (AVDD_PA1), U1.10 (AVDD_PA2), U1.13 (AVDD_LNA), U1.16 (AVDD_BIAS)
- no-connect marks 16 -> 19
Other:
- moved on the sheet: SW1

Commit message: hardware: update gerber file
Parts:
- U2: footprint Housings_DFN_QFN:QFN-48-1EP_7x7mm_Pitch0.5mm -> t3:cc2400_Soldering
Connections:
- net CSn: now also U3.25 (PC5/ADC1_IN15/ADC2_IN15)
- net DCLK: now also U3.26 (ADC1_IN8/ADC2_IN8/TIM1_CH2N/TIM3_CH3/TIM8_CH2N/USB_OTG_HS_ULPI_D1/PB0)
- net DIO: now also U3.27 (ADC1_IN9/ADC2_IN9/TIM1_CH3N/TIM3_CH4/TIM8_CH3N/USB_OTG_HS_ULPI_D2/PB1)
- net SCLK: now also U3.24 (PC4/ADC1_IN14/ADC2_IN14)
- no-connect marks 19 -> 15
Other:
- note added: "!!!"
Changed lines of the file:
@@
 F 0 "U2" H 6400 3100 60  0000 C CNN
 F 1 "CC2400" H 6400 2900 60  0000 C CNN
-F 2 "Housings_DFN_QFN:QFN-48-1EP_7x7mm_Pitch0.5mm" H 6400 3000 60  0001 C CNN
+F 2 "t3:cc2400_Soldering" H 6400 3000 60  0001 C CNN
 F 3 "" H 6400 3000 60  0001 C CNN
 	1    6400 3000
@@
 	0    -1   -1   0
 $EndComp
-NoConn ~ 12850 7900
-NoConn ~ 12850 8000
 $Comp
 L R R12
@@
 NoConn ~ 4250 7900
 NoConn ~ 4250 8000
-NoConn ~ 4250 8300
-NoConn ~ 4250 8400
 NoConn ~ 4250 8800
 NoConn ~ 4250 9100
@@
 Text Label 13900 2550 2    47   Italic 9
 GIO1
+Wire Wire Line
+	4250 8300 3950 8300
+Text Notes 3850 8300 0    60   ~ 0
+!!!
+Text Label 3950 8300 0    39   Italic 8
+SCLK
+Wire Wire Line
+	4250 8400 3950 8400
+Text Notes 3850 8400 0    60   ~ 0
+!!!
+Text Label 3950 8400 0    39   Italic 8
+CSn
+Wire Wire Line
+	12850 7900 13150 7900
+Wire Wire Line
+	12850 8000 13150 8000
+Text Label 13150 7900 2    39   Italic 8
+DCLK
+Text Label 13150 8000 2    39   Italic 8
+DIO
+Text Notes 13150 7900 0    60   ~ 0
+!!!
+Text Notes 13150 8000 0    60   ~ 0
+!!!
 $EndSCHEMATC
