File: hardware/t3/t3.kicad_pcb (KiCad board)
At the start: 2 copper layers, 81.3 x 45.7 mm, 83 parts, among them P1 SMA, P2 CON, P3 UART1, P4 SWD, P5 USB_B, P6 power, P7 UART2, P8 Debug, Q1 9012, SW1 SW_PUSH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

Commit message: hardware: update gerber file
Parts:
- removed the G*** at (114.8, 81.3)
- added G***: LOGO, t3:logo, F.Cu at (114.6, 84.1)
- U2: footprint Housings_DFN_QFN:QFN-48-1EP_7x7mm_Pitch0.5mm -> t3:cc2400_Soldering
- moved U2 4.31 mm to (140.1, 93.4)
- moved C3 3.94 mm to (123.7, 98.2), turned to 90 degrees
- moved C1 3.38 mm to (116.8, 96.3), turned to 270 degrees
- moved P1 3.05 mm to (111.0, 97.3)
- moved L1 2.40 mm to (118.4, 96.3)
- moved L2 1.65 mm to (121.0, 97.3)
- moved t5 1.52 mm to (151.1, 98.0)
- moved t1 0.72 mm to (141.2, 87.4)
Connections:
- U3 pad 24: Net-(U3-Pad24) -> /SCLK
- U3 pad 25: Net-(U3-Pad25) -> /CSn
- U3 pad 26: Net-(U3-Pad26) -> /DCLK
- U3 pad 27: Net-(U3-Pad27) -> /DIO
Routing:
- net GND: track 579.6 -> 662.0 mm, vias 29 -> 102
- net Net-(P4-Pad2): track 41.4 -> 59.2 mm
- net (no net): track 15.2 -> 26.6 mm, vias 16 -> 6
- net /ATEST1: track 10.3 -> 21.1 mm
- net +1V8: track 111.2 -> 118.6 mm
- net /DIO: track 19.7 -> 24.1 mm
- net /CSn: track 8.35 -> 11.9 mm, vias 2 -> 0
- net /SCLK: track 7.22 -> 10.0 mm, vias 2 -> 0
- net Net-(C1-Pad2): track 11.7 -> 9.02 mm
- net /GIO6: track 11.9 -> 13.0 mm
- net /GIO1: track 16.8 -> 15.9 mm
- net /GR: track 16.5 -> 15.7 mm
- net Net-(R11-Pad1): track 7.75 -> 8.31 mm
- net /DCLK: track 20.3 -> 20.2 mm, vias 2 -> 1
Other:
- board size 81.3 x 45.7 mm -> 83.3 x 45.7 mm
- board text added: "Appotech.com"
