File: ubertooth/hardware/ubertooth-one/ubertooth-one.sch (KiCad schematic (older format))
At the start: 89 parts, among them J1 USB-DEVICE, P1 SMA-CONN, P10 ATEST1, P11 ATEST2, P12 DCLK, P13 DIO, P2 PROGRAM, P3 JTAG, P4 EXPAND, P5 1V8, P6 3V3, P7 VBUS, P8 GIO1, P9 GIO6, Q1 BC856, U1 CC2591, U3 CC2400, U4 LPC175X, U6 IP4220CZ6, U7 TPS71219, X1 ABMM2

Commit message: push LPC datasheet
Parts:
- C1, C10, C11, C12, C14, C15, C16, C17, C18, C19, C2, C20, C21, C22, C23, C24, C25, C26, C27, C28, C29, C3, C30, C31, C32, C33, C34, C35, C36, C4, C5, C6, C7, C8, C9: symbol C -> C-RESCUE-ubertooth-one
- D1, D2, D3, D4, D5, D6: symbol LED -> LED-RESCUE-ubertooth-one
- R1, R10, R11, R12, R13, R14, R15, R16, R17, R18, R19, R2, R3, R4, R5, R6, R7, R8, R9: symbol R -> R-RESCUE-ubertooth-one
