File: hardware/v2/ubermini.sch (KiCad schematic (older format))
At the start: 70 parts, among them P1 SMA-CONN, P2 sma, P3 sma, P4 uart1, P5 SWD, P6 boot, P7 USB_B, SW1 SW_PUSH, U1 CC2591, U2 STM32F405RGTx, U3 CC2400, U4 TPS712XX, Y1 16m

Commit message: hw v2 update
Parts:
- removed P7: USB_B, symbol USB_B
- added J1: USB_OTG, Connect:USB_Mini-B, symbol USB_OTG
- added P7: sma, v2:U.FL, symbol CONN_01X02
- BT1: footprint (none) -> Pin_Headers:Pin_Header_Straight_1x02
- C1, C10, C11, C12, C13, C14, C15, C16, C17, C18, C19, C2, C20, C21, C22, C29, C3, C30, C31, C32, C33, C5, C6, C7, L4: footprint (none) -> Capacitors_SMD:C_0603_HandSoldering
- C23: renamed from C24; footprint (none) -> Capacitors_SMD:C_0603_HandSoldering
- C24: renamed from C26; footprint (none) -> Capacitors_SMD:C_0603_HandSoldering
- C25: renamed from C23; footprint (none) -> Capacitors_SMD:C_0603_HandSoldering
- C26: renamed from C28; footprint (none) -> Capacitors_SMD:C_0603_HandSoldering
- C27: renamed from C25; footprint (none) -> Capacitors_SMD:C_0603_HandSoldering
- C28: renamed from C27; footprint (none) -> Capacitors_SMD:C_0603_HandSoldering
- C4, C8, C9, L1, L2, L3: footprint (none) -> Capacitors_SMD:C_0402
- D1: renamed from D2; footprint (none) -> Resistors_SMD:R_0805_HandSoldering
- D2: renamed from D1; footprint (none) -> LEDs:LED_0805
- D3, D4, D5: footprint (none) -> Resistors_SMD:R_0805_HandSoldering
- P1: footprint (none) -> v2:sma
- P2, P3: footprint (none) -> v2:U.FL
- P4, P5: footprint (none) -> Pin_Headers:Pin_Header_Straight_1x03
- P6: footprint (none) -> Pin_Headers:Pin_Header_Straight_2x03
- R1, R10, R11, R12, R13, R14, R2, R3, R4, R5, R6, R7, R8, R9: footprint (none) -> Resistors_SMD:R_0603_HandSoldering
- SW1: footprint (none) -> Buttons_Switches_SMD:SW_SPST_FSMSM
- U1: footprint (none) -> v2:cc2591
- U2: footprint LQFP64 -> Housings_QFP:LQFP-64_10x10mm_Pitch0.5mm
- U3: footprint (none) -> v2:cc2400
- U4: footprint (none) -> v2:tps712
- Y1: footprint (none) -> Crystals:Crystal_SMD_0603_4Pads
Connections:
- wire segments 243 -> 245
Other:
- moved on the sheet: BT1, C23, C24, C26, C32, C33, D1, L4, R10, R9, U4

Commit message: hw v2 add pcb
Parts:
- D3, D4, D5: footprint Resistors_SMD:R_0805_HandSoldering -> LEDs:LED_0805
Connections:
- net CSn: now also U2.54 (PD2/SDIO_CMD/TIM3_ETR/UART5_RX)
- net DCLK: now also U2.55 (I2S3_CK/SPI1_SCK/SPI3_SCK/SYS_JTDO-SWO/TIM2_CH2/PB3)
- net DIO: now also U2.56 (I2S3_ext_SD/SPI1_MISO/SPI3_MISO/SYS_JTRST/TIM3_CH1/PB4), U2.57 (CAN2_RX/I2C1_SMBA/I2S3_SD/SPI1_MOSI/SPI3_MOSI/TIM3_CH2/USB_OTG_HS_ULPI_D7/PB5)
- net GIO6: now also U2.50 (ADC1_EXTI15/ADC2_EXTI15/ADC3_EXTI15/I2S3_WS/SPI1_NSS/SPI3_NSS/SYS_JTDI/TIM2_CH1/TIM2_ETR/PA15)
- net RX: now also U2.59 (I2C1_SDA/TIM4_CH2/USART1_RX/PB7)
- net SCLK: now also U2.53 (PC12/I2S3_SD/SDIO_CK/SPI3_MOSI/UART5_TX/USART3_CK)
- net SI: now also U2.52 (PC11/ADC1_EXTI11/ADC2_EXTI11/ADC3_EXTI11/I2S3_ext_SD/SDIO_D3/SPI3_MISO/UART4_RX/USART3_RX)
- net SO: now also U2.51 (PC10/I2S3_CK/SDIO_D2/SPI3_SCK/UART4_TX/USART3_TX)
- net TX: now also U2.58 (CAN2_TX/I2C1_SCL/TIM4_CH1/USART1_TX/PB6)
Changed lines of the file:
@@
 Text Label 8550 2150 0    60   ~ 0
 ATEST2
-Text Label 15200 5850 2    60   ~ 0
+Text Label 11250 8250 2    60   ~ 0
 GIO6
-Text Label 15150 5950 2    60   ~ 0
+Text Label 1850 9350 2    60   ~ 0
 SO
-Text Label 15150 6050 2    60   ~ 0
+Text Label 1850 9450 2    60   ~ 0
 SI
-Text Label 15150 6150 2    60   ~ 0
+Text Label 1850 9550 2    60   ~ 0
 SCLK
-Text Label 15150 6250 2    60   ~ 0
+Text Label 1900 8150 2    60   ~ 0
 CSn
-Text Label 15200 6400 2    60   ~ 0
+Text Label 11300 8650 2    60   ~ 0
 DCLK
-Text Label 15150 6500 2    60   ~ 0
+Text Label 11300 8750 2    60   ~ 0
 DIO
-Text Label 15150 6650 2    60   ~ 0
+Text Label 11300 8950 2    60   ~ 0
 TX
-Text Label 15150 6800 2    60   ~ 0
+Text Label 11300 9050 2    60   ~ 0
 RX
 $Comp
@@
 F 0 "D3" H 14250 3900 50  0000 C CNN
 F 1 "LED" H 14400 3900 50  0000 C CNN
-F 2 "Resistors_SMD:R_0805_HandSoldering" H 14250 3800 50  0001 C CNN
+F 2 "LEDs:LED_0805" H 14250 3800 50  0001 C CNN
 F 3 "" H 14250 3800 50  0000 C CNN
 	1    14250 3800
@@
 F 0 "D4" H 14450 3900 50  0000 C CNN
 F 1 "LED" H 14600 3900 50  0000 C CNN
-F 2 "Resistors_SMD:R_0805_HandSoldering" H 14450 3800 50  0001 C CNN
+F 2 "LEDs:LED_0805" H 14450 3800 50  0001 C CNN
 F 3 "" H 14450 3800 50  0000 C CNN
 	1    14450 3800
@@
 F 0 "D5" H 14650 3900 50  0000 C CNN
 F 1 "LED" H 14800 3900 50  0000 C CNN
-F 2 "Resistors_SMD:R_0805_HandSoldering" H 14650 3800 50  0001 C CNN
+F 2 "LEDs:LED_0805" H 14650 3800 50  0001 C CNN
 F 3 "" H 14650 3800 50  0000 C CNN
 	1    14650 3800
@@
 	1    12200 7850
 	-1   0    0    1
+$EndComp
+$Comp
+L GND #PWR039
+U 1 1 5900F50A
+P 12200 7200
+F 0 "#PWR039" H 12200 6950 50  0001 C CNN
+F 1 "GND" H 12200 7050 50  0000 C CNN
+F 2 "" H 12200 7200 50  0000 C CNN
+F 3 "" H 12200 7200 50  0000 C CNN
+	1    12200 7200
+	-1   0    0    1
+$EndComp
+$Comp
+L CONN_01X02 P7
+U 1 1 590260DB
+P 1950 4150
+F 0 "P7" H 1950 4300 50  0000 C CNN
+F 1 "sma" V 2050 4150 50  0000 C CNN
+F 2 "v2:U.FL" H 1950 4150 50  0001 C CNN
+F 3 "" H 1950 4150 50  0000 C CNN
+	1    1950 4150
+	0    -1   1    0
 $EndComp
 Wire Wire Line
@@
 	11850 7650 11900 7650
 Connection ~ 12200 7250
-$Comp
-L GND #PWR039
-U 1 1 5900F50A
-P 12200 7200
-F 0 "#PWR039" H 12200 6950 50  0001 C CNN
-F 1 "GND" H 12200 7050 50  0000 C CNN
-F 2 "" H 12200 7200 50  0000 C CNN
-F 3 "" H 12200 7200 50  0000 C CNN
-	1    12200 7200
-	-1   0    0    1
-$EndComp
 Wire Wire Line
 	1750 7850 1550 7850
@@
 	1550 7850 1550 8150
 Connection ~ 7250 1300
-$Comp
-L CONN_01X02 P7
-U 1 1 590260DB
-P 1950 4150
-F 0 "P7" H 1950 4300 50  0000 C CNN
-F 1 "sma" V 2050 4150 50  0000 C CNN
-F 2 "v2:U.FL" H 1950 4150 50  0001 C CNN
-F 3 "" H 1950 4150 50  0000 C CNN
-	1    1950 4150
-	0    -1   1    0
-$EndComp
 Connection ~ 2000 3950
 Wire Wire Line
 	1900 3950 1900 3500
 Connection ~ 1900 3500
+Wire Wire Line
+	10750 8750 11300 8750
+Wire Wire Line
+	11050 8750 11050 8850
+Wire Wire Line
+	11050 8850 10750 8850
+Connection ~ 11050 8750
+Wire Wire Line
+	10750 8650 11300 8650
+Wire Wire Line
+	2150 8150 1900 8150
+Wire Wire Line
+	2150 9350 1850 9350
+Wire Wire Line
+	2150 9450 1850 9450
+Wire Wire Line
+	2150 9550 1850 9550
+Wire Wire Line
+	10750 8150 10750 8250
+Wire Wire Line
+	10750 8250 11250 8250
+Wire Wire Line
+	10750 8950 11300 8950
+Wire Wire Line
+	10750 9050 11300 9050
 $EndSCHEMATC

Commit message: hw update
Connections:
- net +3.3VA: no longer U4.7 (FB2/NC)
- net GR: now also U2.61 (CAN1_RX/I2C1_SCL/SDIO_D4/TIM10_CH1/TIM4_CH3/PB8)
- net LED1: now also U2.8 (PC0/ADC1_IN10/ADC2_IN10/ADC3_IN10/USB_OTG_HS_ULPI_STP)
- net LED2: now also U2.9 (PC1/ADC1_IN11/ADC2_IN11/ADC3_IN11)
- net LED3: now also U2.10 (PC2/ADC1_IN12/ADC2_IN12/ADC3_IN12/I2S2_ext_SD/SPI2_MISO/USB_OTG_HS_ULPI_DIR)
- net LED4: now also U2.11 (PC3/ADC1_IN13/ADC2_IN13/ADC3_IN13/I2S2_SD/SPI2_MOSI/USB_OTG_HS_ULPI_NXT)
- net SPI1_CS: now reaches U2.20 (ADC1_IN4/ADC2_IN4/DAC_OUT1/I2S3_WS/SPI1_NSS/SPI3_NSS/USART2_CK/USB_OTG_HS_SOF/PA4)
- net SPI1_SCK: now reaches U2.21 (ADC1_IN5/ADC2_IN5/DAC_OUT2/SPI1_SCK/TIM2_CH1/TIM2_ETR/TIM8_CH1N/USB_OTG_HS_ULPI_CK/PA5)
- net SPI1_MI: now reaches U2.22 (ADC1_IN6/ADC2_IN6/SPI1_MISO/TIM13_CH1/TIM1_BKIN/TIM3_CH1/TIM8_BKIN/PA6)
- net SPI1_MO: now reaches U2.23 (ADC1_IN7/ADC2_IN7/SPI1_MOSI/TIM14_CH1/TIM1_CH1N/TIM3_CH2/TIM8_CH1N/PA7)
- net at C33.2, R10.1, R9.2: now also U4.7 (FB2/NC)
- net ATEST1 renamed ATEST1_P
- net ATEST2 renamed ATEST2_N
Changed lines of the file:
@@
 $EndComp
 Text Label 6800 1400 3    60   ~ 0
-ATEST1
+ATEST1_P
 Text Label 6900 1400 3    60   ~ 0
-ATEST2
+ATEST2_N
 $Comp
 L Crystal_GND24 Y1
@@
 Text Label 15000 7000 3    60   ~ 0
 EN
-Text Label 15150 7100 1    60   ~ 0
+Text Label 11300 9150 2    60   ~ 0
 GR
 Text Label 1550 8150 1    60   ~ 0
 GIO1
 Text Label 8550 1700 0    60   ~ 0
-ATEST1
+ATEST1_P
 Text Label 8550 2150 0    60   ~ 0
-ATEST2
+ATEST2_N
 Text Label 11250 8250 2    60   ~ 0
 GIO6
@@
 Connection ~ 13150 1450
 Wire Wire Line
-	13050 1750 13600 1750
-Wire Wire Line
 	13600 1750 13600 1800
 Wire Wire Line
@@
 Connection ~ 13400 1750
 Wire Wire Line
-	13600 2100 13600 2150
-Wire Wire Line
-	13600 2150 13400 2150
+	13600 2150 13600 2100
+Wire Wire Line
+	13250 2150 13600 2150
 Wire Wire Line
 	13400 2100 13400 2200
@@
 Wire Wire Line
 	10750 9050 11300 9050
+Text Label 1900 8350 0    60   ~ 0
+LED1
+Wire Wire Line
+	1900 8350 2150 8350
+Wire Wire Line
+	2150 8450 1900 8450
+Wire Wire Line
+	2150 8550 1900 8550
+Wire Wire Line
+	2150 8650 1900 8650
+Text Label 1900 8450 0    60   ~ 0
+LED2
+Text Label 1900 8550 0    60   ~ 0
+LED3
+Text Label 1900 8650 0    60   ~ 0
+LED4
+Wire Wire Line
+	10750 7050 11000 7050
+Wire Wire Line
+	10750 7150 11000 7150
+Wire Wire Line
+	10750 7250 11000 7250
+Wire Wire Line
+	10750 7350 11000 7350
+Text Label 11000 7050 0    60   ~ 0
+SPI1_CS
+Text Label 11000 7150 0    60   ~ 0
+SPI1_SCK
+Text Label 11000 7250 0    60   ~ 0
+SPI1_MI
+Text Label 11000 7350 0    60   ~ 0
+SPI1_MO
+Wire Wire Line
+	13400 1750 13600 1750
+Wire Wire Line
+	13050 1750 13250 1750
+Wire Wire Line
+	13250 1750 13250 2150
+Wire Wire Line
+	10750 9150 11300 9150
 $EndSCHEMATC

Commit message: hw update
Parts:
- added D6: LED, LEDs:LED_0805, symbol LED
- added R15: 10k, Resistors_SMD:R_0603_HandSoldering, symbol R
- added U5: M25PX32-VMW, v2:winband_spi_flash, symbol M25PX32-VMW
Connections:
- net +3V3: now also D6.2 (A), U5.3 (W#/VPP), U5.7 (HOLD#), U5.8 (VCC)
- net EN: now also U2.3 (PC14/RCC_OSC32_IN)
- net GND: now also R15.2, U5.4 (VSS)
- net HGM: now also U2.4 (PC15/ADC1_EXTI15/ADC2_EXTI15/ADC3_EXTI15/RCC_OSC32_OUT)
- net SPI1_CS: now also U5.1 (S#); no longer U2.20 (ADC1_IN4/ADC2_IN4/DAC_OUT1/I2S3_WS/SPI1_NSS/SPI3_NSS/USART2_CK/USB_OTG_HS_SOF/PA4)
- net SPI1_MI: now also U5.2 (DQ1)
- net SPI1_MO: now also U5.5 (DQ0)
- net SPI1_SCK: now also U5.6 (C)
- new net: D6.1 (K), R15.1
- no-connect marks 11 -> 34
Changed lines of the file:
@@
 	0    1    1    0
 $EndComp
-Text Label 14800 6950 3    60   ~ 0
+Text Label 1850 9850 0    60   ~ 0
 HGM
-Text Label 15000 7000 3    60   ~ 0
+Text Label 1850 9750 0    60   ~ 0
 EN
 Text Label 11300 9150 2    60   ~ 0
@@
 	0    -1   1    0
 $EndComp
+Text Label 1900 8350 0    60   ~ 0
+LED1
+Text Label 1900 8450 0    60   ~ 0
+LED2
+Text Label 1900 8550 0    60   ~ 0
+LED3
+Text Label 1900 8650 0    60   ~ 0
+LED4
+Text Label 12250 6200 0    60   ~ 0
+SPI1_CS
+Text Label 11000 7150 0    60   ~ 0
+SPI1_SCK
+Text Label 11000 7250 0    60   ~ 0
+SPI1_MI
+Text Label 11000 7350 0    60   ~ 0
+SPI1_MO
+$Comp
+L R R15
+U 1 1 5914A2C3
+P 14950 2350
+F 0 "R15" V 15030 2350 50  0000 C CNN
+F 1 "10k" V 14950 2350 50  0000 C CNN
+F 2 "Resistors_SMD:R_0603_HandSoldering" V 14880 2350 50  0001 C CNN
+F 3 "" H 14950 2350 50  0000 C CNN
+	1    14950 2350
+	1    0    0    -1
+$EndComp
+$Comp
+L LED D6
+U 1 1 5914A2C9
+P 14950 2000
+F 0 "D6" H 14950 2100 50  0000 C CNN
+F 1 "LED" H 15100 2100 50  0000 C CNN
+F 2 "LEDs:LED_0805" H 14950 2000 50  0001 C CNN
+F 3 "" H 14950 2000 50  0000 C CNN
+	1    14950 2000
+	0    -1   -1   0
+$EndComp
+$Comp
+L GND #PWR040
+U 1 1 59161DFC
+P 14950 2600
+F 0 "#PWR040" H 14950 2350 50  0001 C CNN
+F 1 "GND" H 14950 2450 50  0000 C CNN
+F 2 "" H 14950 2600 50  0000 C CNN
+F 3 "" H 14950 2600 50  0000 C CNN
+	1    14950 2600
+	1    0    0    -1
+$EndComp
+$Comp
+L +3.3V #PWR041
+U 1 1 5916261F
+P 14950 1600
+F 0 "#PWR041" H 14950 1450 50  0001 C CNN
+F 1 "+3.3V" H 14950 1740 50  0000 C CNN
+F 2 "" H 14950 1600 50  0000 C CNN
+F 3 "" H 14950 1600 50  0000 C CNN
+	1    14950 1600
+	1    0    0    -1
+$EndComp
+$Comp
+L M25PX32-VMW U5
+U 1 1 59163808
+P 13300 6200
+F 0 "U5" H 12900 6600 50  0000 C CNN
+F 1 "M25PX32-VMW" H 13600 5800 50  0000 C CNN
+F 2 "v2:winband_spi_flash" H 13950 6250 50  0001 C CNN
+F 3 "" H 13450 6100 50  0001 C CNN
+	1    13300 6200
+	1    0    0    -1
+$EndComp
 Wire Wire Line
 	4050 1500 4050 2550
@@
 Wire Wire Line
 	10750 9050 11300 9050
-Text Label 1900 8350 0    60   ~ 0
-LED1
 Wire Wire Line
 	1900 8350 2150 8350
@@
 Wire Wire Line
 	2150 8650 1900 8650
-Text Label 1900 8450 0    60   ~ 0
-LED2
-Text Label 1900 8550 0    60   ~ 0
-LED3
-Text Label 1900 8650 0    60   ~ 0
-LED4
 Wire Wire Line
 	10750 7050 11000 7050
@@
 Wire Wire Line
 	10750 7350 11000 7350
-Text Label 11000 7050 0    60   ~ 0
-SPI1_CS
-Text Label 11000 7150 0    60   ~ 0
+Wire Wire Line
+	13400 1750 13600 1750
+Wire Wire Line
+	13050 1750 13250 1750
+Wire Wire Line
+	13250 1750 13250 2150
+Wire Wire Line
+	10750 9150 11300 9150
+Wire Wire Line
+	14950 2500 14950 2600
+Wire Wire Line
+	14950 2150 14950 2200
+Wire Wire Line
+	14950 1850 14950 1600
+Wire Wire Line
+	2150 9850 1850 9850
+Wire Wire Line
+	2150 9750 1850 9750
+Wire Wire Line
+	12250 6000 12700 6000
+Wire Wire Line
+	12250 6100 12700 6100
+Wire Wire Line
+	12250 6200 12700 6200
+Wire Wire Line
+	12700 6300 12450 6300
+Wire Wire Line
+	12450 6300 12450 6400
+Wire Wire Line
+	12450 6400 12700 6400
+$Comp
+L +3.3V #PWR042
+U 1 1 59165267
+P 12450 6350
+F 0 "#PWR042" H 12450 6200 50  0001 C CNN
+F 1 "+3.3V" H 12450 6490 50  0000 C CNN
+F 2 "" H 12450 6350 50  0000 C CNN
+F 3 "" H 12450 6350 50  0000 C CNN
+	1    12450 6350
+	0    -1   -1   0
+$EndComp
+Connection ~ 12450 6350
+$Comp
+L GND #PWR043
+U 1 1 591659C9
+P 13300 6800
+F 0 "#PWR043" H 13300 6550 50  0001 C CNN
+F 1 "GND" H 13300 6650 50  0000 C CNN
+F 2 "" H 13300 6800 50  0000 C CNN
+F 3 "" H 13300 6800 50  0000 C CNN
+	1    13300 6800
+	1    0    0    -1
+$EndComp
+Wire Wire Line
+	13300 6800 13300 6700
+$Comp
+L +3.3V #PWR044
+U 1 1 591660EE
+P 13300 5650
+F 0 "#PWR044" H 13300 5500 50  0001 C CNN
+F 1 "+3.3V" H 13300 5790 50  0000 C CNN
+F 2 "" H 13300 5650 50  0000 C CNN
+F 3 "" H 13300 5650 50  0000 C CNN
+	1    13300 5650
+	1    0    0    -1
+$EndComp
+Wire Wire Line
+	13300 5700 13300 5650
+Wire Wire Line
+	13900 6000 14250 6000
+Text Label 12250 6100 0    60   ~ 0
 SPI1_SCK
-Text Label 11000 7250 0    60   ~ 0
+Text Label 12250 6000 0    60   ~ 0
+SPI1_MO
+Text Label 14250 6000 2    60   ~ 0
 SPI1_MI
-Text Label 11000 7350 0    60   ~ 0
-SPI1_MO
-Wire Wire Line
-	13400 1750 13600 1750
-Wire Wire Line
-	13050 1750 13250 1750
-Wire Wire Line
-	13250 1750 13250 2150
-Wire Wire Line
-	10750 9150 11300 9150
+NoConn ~ 2150 8750
+NoConn ~ 2150 8850
+NoConn ~ 2150 8950
+NoConn ~ 2150 9050
+NoConn ~ 2150 9150
+NoConn ~ 2150 9250
+NoConn ~ 2150 9650
+NoConn ~ 11000 7050
+NoConn ~ 10750 9250
+NoConn ~ 10750 9350
+NoConn ~ 10750 9450
+NoConn ~ 10750 9550
+NoConn ~ 10750 9650
+NoConn ~ 10750 9750
+NoConn ~ 10750 9850
+NoConn ~ 10750 8450
+NoConn ~ 10750 8350
+NoConn ~ 10750 7450
+NoConn ~ 10750 6950
+NoConn ~ 10750 6850
+NoConn ~ 10750 6750
+NoConn ~ 10750 6650
+NoConn ~ 2150 7950
 $EndSCHEMATC

Commit message: hw update
Parts:
- D2, D3, D4, D5, D6: symbol LED -> LED-RESCUE-ubermini
- J1: footprint Connect:USB_Mini-B -> v2:USB_Mini-B_s; symbol USB_OTG -> USB_OTG-RESCUE-ubermini
Connections:
- net EN: now also U2.2 (PC13/ANTI_TAMP/RTC_AF1); no longer U2.3 (PC14/RCC_OSC32_IN)
- net HGM: now also U2.3 (PC14/RCC_OSC32_IN); no longer U2.4 (PC15/ADC1_EXTI15/ADC2_EXTI15/ADC3_EXTI15/RCC_OSC32_OUT)
- net SPI1_CS: now also U2.4 (PC15/ADC1_EXTI15/ADC2_EXTI15/ADC3_EXTI15/RCC_OSC32_OUT)
- no-connect marks 34 -> 33
Changed lines of the file:
@@
 EESchema Schematic File Version 2
+LIBS:ubermini-rescue
 LIBS:power
 LIBS:device
@@
 	0    1    1    0
 $EndComp
-Text Label 1850 9850 0    60   ~ 0
+Text Label 1850 9750 0    60   ~ 0
 HGM
-Text Label 1850 9750 0    60   ~ 0
+Text Label 1850 9650 0    60   ~ 0
 EN
 Text Label 11300 9150 2    60   ~ 0
@@
 $EndComp
 $Comp
-L LED D2
+L LED-RESCUE-ubermini D2
 U 1 1 58FFDCAF
 P 14050 3800
@@
 $EndComp
 $Comp
-L LED D3
+L LED-RESCUE-ubermini D3
 U 1 1 58FFE046
 P 14250 3800
@@
 $EndComp
 $Comp
-L LED D4
+L LED-RESCUE-ubermini D4
 U 1 1 58FFE123
 P 14450 3800
@@
 $EndComp
 $Comp
-L LED D5
+L LED-RESCUE-ubermini D5
 U 1 1 58FFE207
 P 14650 3800
@@
 $EndComp
 $Comp
-L USB_OTG J1
+L USB_OTG-RESCUE-ubermini J1
 U 1 1 5900CA0C
 P 12200 7850
 F 0 "J1" H 12000 8300 50  0000 L CNN
 F 1 "USB_OTG" H 12000 8200 50  0000 L CNN
-F 2 "Connect:USB_Mini-B" H 12350 7800 50  0001 C CNN
+F 2 "v2:USB_Mini-B_s" H 12350 7800 50  0001 C CNN
 F 3 "" H 12350 7800 50  0001 C CNN
 	1    12200 7850
@@
 $EndComp
 $Comp
-L LED D6
+L LED-RESCUE-ubermini D6
 U 1 1 5914A2C9
 P 14950 2000
@@
 NoConn ~ 2150 9150
 NoConn ~ 2150 9250
-NoConn ~ 2150 9650
 NoConn ~ 11000 7050
 NoConn ~ 10750 9250
@@
 NoConn ~ 10750 6650
 NoConn ~ 2150 7950
+Wire Wire Line
+	2150 9650 1850 9650
+Text Label 1850 9850 0    60   ~ 0
+SPI1_CS
 $EndSCHEMATC

Commit message: add logo
Parts:
- Y1: footprint Crystals:Crystal_SMD_0603_4Pads -> v2:3225
Changed lines of the file:
@@
 F 0 "Y1" H 7250 1700 50  0000 L CNN
 F 1 "16m" H 7300 1600 50  0000 L CNN
-F 2 "Crystals:Crystal_SMD_0603_4Pads" H 7250 1500 50  0001 C CNN
+F 2 "v2:3225" H 7250 1500 50  0001 C CNN
 F 3 "" H 7250 1500 50  0000 C CNN
 	1    7250 1500

Commit message: create gerber file
Parts:
- C7: value 18nF -> 18pF
Changed lines of the file:
@@
 P 2650 3200
 F 0 "C7" H 2675 3300 50  0000 L CNN
-F 1 "18nF" H 2675 3100 50  0000 L CNN
+F 1 "18pF" H 2675 3100 50  0000 L CNN
 F 2 "Capacitors_SMD:C_0603_HandSoldering" H 2688 3050 50  0001 C CNN
 F 3 "" H 2650 3200 50  0000 C CNN

Commit message: upload pcb n2
Parts:
- added F1, F2, F3: 0, Capacitors_SMD:C_0201, symbol R
- L1, L2: footprint Capacitors_SMD:C_0402 -> Capacitors_SMD:C_0603
Connections:
- net +1V8: now also F1.1; no longer U4.3 (OUT1)
- net +3.3VA: now also F2.1; no longer U4.4 (OUT2)
- net at C4.2, L1.2, L2.1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: now also F3.1; no longer P7.1 (P1)
- new net: F1.2, U4.3 (OUT1)
- new net: F2.2, U4.4 (OUT2)
- new net: F3.2, P7.1 (P1)
Changed lines of the file:
@@
 F 0 "L2" V 2300 3400 50  0000 C CNN
 F 1 "2n2" V 2300 3600 50  0000 C CNN
-F 2 "Capacitors_SMD:C_0402" H 2350 3500 50  0001 C CNN
+F 2 "Capacitors_SMD:C_0603" H 2350 3500 50  0001 C CNN
 F 3 "" H 2350 3500 50  0000 C CNN
 	1    2350 3500
@@
 F 0 "L1" V 1950 3200 50  0000 C CNN
 F 1 "3nH" V 1950 3400 50  0000 C CNN
-F 2 "Capacitors_SMD:C_0402" H 2000 3300 50  0001 C CNN
+F 2 "Capacitors_SMD:C_0603" H 2000 3300 50  0001 C CNN
 F 3 "" H 2000 3300 50  0000 C CNN
 	1    2000 3300
@@
 P 2000 3750
 F 0 "C4" V 2050 3800 50  0000 L CNN
-F 1 "2p2" V 2150 3700 50  0000 L CNN
+F 1 "2p2" V 1850 3700 50  0000 L CNN
 F 2 "Capacitors_SMD:C_0402" H 2038 3600 50  0001 C CNN
 F 3 "" H 2000 3750 50  0000 C CNN
@@
 	11000 1450 11000 1800
 Wire Wire Line
-	11750 1650 11250 1650
-Wire Wire Line
 	11250 1200 11250 1800
 Connection ~ 11250 1650
-Wire Wire Line
-	11750 1750 11500 1750
 Wire Wire Line
 	11500 1200 11500 1800
@@
 Connection ~ 7250 1300
 Connection ~ 2000 3950
-Wire Wire Line
-	1900 3950 1900 3500
 Connection ~ 1900 3500
 Wire Wire Line
@@
 Text Label 1850 9850 0    60   ~ 0
 SPI1_CS
+$Comp
+L R F1
+U 1 1 592BE45F
+P 11450 1650
+F 0 "F1" V 11550 1650 50  0000 C CNN
+F 1 "0" V 11450 1650 50  0000 C CNN
+F 2 "Capacitors_SMD:C_0201" V 11380 1650 50  0001 C CNN
+F 3 "" H 11450 1650 50  0000 C CNN
+	1    11450 1650
+	0    -1   -1   0
+$EndComp
+$Comp
+L R F2
+U 1 1 592BF4BE
+P 11550 1750
+F 0 "F2" V 11500 1600 50  0000 C CNN
+F 1 "0" V 11550 1750 50  0000 C CNN
+F 2 "Capacitors_SMD:C_0201" V 11480 1750 50  0001 C CNN
+F 3 "" H 11550 1750 50  0000 C CNN
+	1    11550 1750
+	0    -1   -1   0
+$EndComp
+Wire Wire Line
+	11600 1650 11750 1650
+Wire Wire Line
+	11250 1650 11300 1650
+Wire Wire Line
+	11700 1750 11750 1750
+Wire Wire Line
+	11500 1750 11400 1750
+$Comp
+L R F3
+U 1 1 592C70A9
+P 1850 3750
+F 0 "F3" V 1750 3750 50  0000 C CNN
+F 1 "0" V 1850 3750 50  0000 C CNN
+F 2 "Capacitors_SMD:C_0201" V 1780 3750 50  0001 C CNN
+F 3 "" H 1850 3750 50  0000 C CNN
+	1    1850 3750
+	1    0    0    -1
+$EndComp
+Wire Wire Line
+	1900 3500 1900 3600
+Wire Wire Line
+	1900 3600 1850 3600
+Wire Wire Line
+	1850 3900 1900 3900
+Wire Wire Line
+	1900 3900 1900 3950
 $EndSCHEMATC
